File: hardware/mainboard/mainboard.kicad_pcb (KiCad board)
At the start: 2 copper layers, 9.2 x 110.3 mm, 8 parts, among them J1 IN1, J2 OUT1, J3 OUT2, J4 OUT3, J5 IN2, J6 OUT4, J7 OUT5, J8 OUT6

Commit message: Update mainboard
Routing:
- net GROUP_1: track 0.00 -> 60.2 mm
- net GROUP_2: track 0.00 -> 51.6 mm
- added copper zone on F.Cu, net GND
- removed copper zone on F.Cu, net GROUP_1
- removed copper zone on F.Cu, net GROUP_2
